Commit message: Add gripper TCP frame for Piper X

File: piper_x/urdf/piper_x_with_gripper_description.xacro (robot description, xacro)
@@ -27,4 +27,11 @@
         <parent link="link6"/>
         <child link="gripper_base"/>
+    </joint>
+    <!-- Fixed TCP frame used as the grasp reference point. -->
+    <link name="gripper_tcp"/>
+    <joint name="gripper_tcp_joint" type="fixed">
+        <origin xyz="0 0 0.1058" rpy="0 0 0"/>
+        <parent link="gripper_base"/>
+        <child link="gripper_tcp"/>
     </joint>
     <link name="gripper_link1">
